File: deska/final/board.brd (EAGLE design)
At the start: 83.7 x 153 mm, 86 parts, among them IC1 DSPIC33EP256MU806-X_PT, IC2 TP4056, SW1 KSS-2EG4430, SW2 KSS-2EG4430, SW3 KSS-2EG4430, U1 TPS731, X1 MINI-USB-UX60-MB-5ST

Commit message: doplneni priloh
Connections:
- new net CH_EN: IC1.6, IC2.8
- net +5V: no longer IC2.8
- net VBAT: now also IC1.11
Routing:
- net +5V: track 29.9 -> 25.9 mm
Changed lines of the file:
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@@
 <contactref element="X1" pad="1"/>
 <contactref element="IC2" pad="4"/>
-<contactref element="IC2" pad="8"/>
 <contactref element="R8" pad="2"/>
 <contactref element="R9" pad="2"/>
@@
 <wire x1="37.789" y1="101.572" x2="37.768" y2="101.551" width="0.508" layer="1"/>
 <wire x1="27.96575" y1="93.7445" x2="30.093" y2="93.7445" width="0.254" layer="1"/>
-<wire x1="32.268" y1="97.741" x2="32.268" y2="95.26" width="0.254" layer="1"/>
 <wire x1="32.268" y1="95.26" x2="30.734" y2="93.726" width="0.254" layer="1"/>
 <wire x1="30.734" y1="93.726" x2="30.1115" y2="93.726" width="0.254" layer="1"/>
@@
 <wire x1="37.789" y1="101.572" x2="37.789" y2="102.803" width="0.6985" layer="1"/>
 <wire x1="37.789" y1="102.803" x2="37.468" y2="103.124" width="0.6985" layer="1"/>
-<wire x1="32.268" y1="97.741" x2="32.268" y2="96.276" width="0.254" layer="1"/>
 <wire x1="32.268" y1="96.276" x2="32.258" y2="96.266" width="0.254" layer="1"/>
 <wire x1="32.258" y1="96.266" x2="36.068" y2="96.266" width="0.254" layer="1"/>
@@
 <wire x1="37.722" y1="103.502" x2="36.068" y2="105.156" width="0.254" layer="1"/>
 <wire x1="36.068" y1="105.156" x2="36.068" y2="96.266" width="0.254" layer="16"/>
+<wire x1="32.268" y1="95.26" x2="32.268" y2="96.276" width="0" layer="19" extent="1-1"/>
 </signal>
 <signal name="VBAT">
@@
 <wire x1="10.922" y1="120.80875" x2="10.922" y2="118.03975" width="0.6985" layer="1"/>
 <wire x1="10.922" y1="118.03975" x2="11.03625" y2="117.9255" width="0.6985" layer="1"/>
+<contactref element="IC1" pad="11"/>
+<wire x1="23.0669" y1="17.0219" x2="23.876" y2="67.818" width="0" layer="19" extent="1-16"/>
 </signal>
 <signal name="+3.15">
@@
 <wire x1="16.6409" y1="10.1639" x2="16.383" y2="9.906" width="0.254" layer="1"/>
 </signal>
+<signal name="CH_EN">
+<contactref element="IC2" pad="8"/>
+<contactref element="IC1" pad="6"/>
+<wire x1="25.5561" y1="17.0219" x2="32.268" y2="97.741" width="0" layer="19" extent="1-1"/>
+</signal>
 </signals>
